File: C4 compact/Bonsai_C4.kicad_pcb (KiCad board)
At the start: 4 copper layers, 17.8 x 33.8 mm, 56 parts, among them J1 HEADER-VERT_3P-2.54_, J14 PAD_SQUARE_1MM, J15 PAD_SQUARE_1MM, J16 PAD_SQUARE_1MM, J2 HEADER-VERT_1P-2.54_, J3 TYPE-C-31-M12_13, J4 HEADER-VERT_12P-2.54_, J5 HEADER-VERT_12P-2.54_, J8 PAD_SQUARE_1MM, K1 SMD-SWITCH-TACTILE-SPST-NO_4P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

Commit message: Added JLCPCB build files for C4, modified C3 JLCPCB files, added schematic notes, updated readmes
Routing:
- net +3V3: track 76.8 -> 75.8 mm
Other:
- board text added: "Bonsai C4 customMK"
