File: C3/Bonsai_C.kicad_pcb (KiCad board)
At the start: 4 copper layers, 17.8 x 51.6 mm, 47 parts, among them J1 HEADER-VERT_3P-2.54_, J10 PAD_SQUARE_1MM, J11 PAD_SQUARE_1MM, J12 PAD_SQUARE_1MM, J14 PAD_SQUARE_1MM, J15 PAD_SQUARE_1MM, J16 PAD_SQUARE_1MM, J2 HEADER-VERT_1P-2.54_, J3 TYPE-C-31-M12_13, J4 HEADER-VERT_12P-2.54_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

Commit message: corrected part number for 0402 capacitor in Bonsai C3 (was 0603 part with 0402 footprint)
Parts:
- C12: value cap_10uF_10v_0402 -> cap_10uF_6v_0402
